File: pcb/driver-v0/blisplay-driver.sch (KiCad schematic (older format))
At the start: 16 parts, among them J1 Conn_01x06, J2 Conn_01x03, J3 Conn_01x03, J4 Conn_01x03, J5 Conn_01x03, J6 Conn_01x03, J7 Conn_01x01, J8 Conn_01x01, U1 74HC595, U11 ULN2803A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

Commit message: Make possible to read driver board with new KiCAD
Not much effort to convert, as this is going to go anyway.
Parts:
- C1, C2: symbol device:C -> blisplay-driver-rescue:C-device
- D1: symbol device:LED -> blisplay-driver-rescue:LED-device
- J1: symbol Connector:Conn_01x06 -> blisplay-driver-rescue:Conn_01x06-Connector
- J2, J3, J4, J5, J6: symbol Connector:Conn_01x03 -> blisplay-driver-rescue:Conn_01x03-Connector
- J7, J8: symbol Connector:Conn_01x01 -> blisplay-driver-rescue:Conn_01x01-Connector
- R1: symbol device:R -> blisplay-driver-rescue:R-device
- U1, U2: symbol Logic_74xx:74HC595 -> blisplay-driver-rescue:74HC595-Logic_74xx
- U11, U21: symbol interface:ULN2803A -> blisplay-driver-rescue:ULN2803A-interface
Changed lines of the file:
@@
 EESchema Schematic File Version 4
-LIBS:blisplay-interface-cache
-EELAYER 28 0
+LIBS:blisplay-driver-cache
+EELAYER 29 0
 EELAYER END
 $Descr A4 11693 8268
@@
 $EndDescr
 $Comp
-L interface:ULN2803A U21
+L blisplay-driver-rescue:ULN2803A-interface U21
 U 1 1 5BCA4A44
 P 4050 4750
@@
 $EndComp
 $Comp
-L interface:ULN2803A U11
+L blisplay-driver-rescue:ULN2803A-interface U11
 U 1 1 5BCA59BE
 P 4000 2550
@@
 $EndComp
 $Comp
-L Logic_74xx:74HC595 U2
+L blisplay-driver-rescue:74HC595-Logic_74xx U2
 U 1 1 5BCAB656
 P 2800 4850
@@
 $EndComp
 $Comp
-L Logic_74xx:74HC595 U1
+L blisplay-driver-rescue:74HC595-Logic_74xx U1
 U 1 1 5BCABF0D
 P 2750 2650
@@
 $EndComp
 $Comp
-L Connector:Conn_01x06 J1
+L blisplay-driver-rescue:Conn_01x06-Connector J1
 U 1 1 5BCBBB09
 P 1250 3750
@@
 carry
 $Comp
-L device:C C1
+L blisplay-driver-rescue:C-device C1
 U 1 1 5BCF7DDB
 P 6300 2800
@@
 	2300 5050 2300 5100
 $Comp
-L device:C C2
+L blisplay-driver-rescue:C-device C2
 U 1 1 5BD64E2D
 P 6050 2800
@@
 	1450 4050 1600 4050
 $Comp
-L Connector:Conn_01x03 J2
+L blisplay-driver-rescue:Conn_01x03-Connector J2
 U 1 1 5BCCEB4F
 P 5450 4950
@@
 $EndComp
 $Comp
-L Connector:Conn_01x03 J3
+L blisplay-driver-rescue:Conn_01x03-Connector J3
 U 1 1 5BCD02A1
 P 5450 4350
@@
 $EndComp
 $Comp
-L Connector:Conn_01x03 J4
+L blisplay-driver-rescue:Conn_01x03-Connector J4
 U 1 1 5BCD08F2
 P 5350 3200
@@
 $EndComp
 $Comp
-L Connector:Conn_01x03 J5
+L blisplay-driver-rescue:Conn_01x03-Connector J5
 U 1 1 5BCD15D5
 P 5350 2750
@@
 $EndComp
 $Comp
-L Connector:Conn_01x03 J6
+L blisplay-driver-rescue:Conn_01x03-Connector J6
 U 1 1 5BCD1FA6
 P 5350 2350
@@
 	4650 3100 5150 3100
 $Comp
-L device:LED D1
+L blisplay-driver-rescue:LED-device D1
 U 1 1 5BD39E39
 P 3500 1950
@@
 $EndComp
 $Comp
-L device:R R1
+L blisplay-driver-rescue:R-device R1
 U 1 1 5BD3C356
 P 3250 2100
@@
 	3650 1950 3650 2000
 $Comp
-L Connector:Conn_01x01 J7
+L blisplay-driver-rescue:Conn_01x01-Connector J7
 U 1 1 5BD4C259
 P 6050 3600
@@
 $EndComp
 $Comp
-L Connector:Conn_01x01 J8
+L blisplay-driver-rescue:Conn_01x01-Connector J8
 U 1 1 5BD5496C
 P 6050 3900
